Commit message: Add materials and colors as used in Agilus-2 series

File: kuka_resources/urdf/common_colours.xacro (robot description, xacro)
@@ -72,5 +72,9 @@
   <!-- RAL 9002 - gray white  -->
   <xacro:property name="colour_kuka_ral_gray_white"       value="${215/255} ${213/255} ${203/255} 1.0" />
+  <!-- RAL 9007 - grey aluminium -->
+  <xacro:property name="colour_kuka_ral_gray_aluminium"   value="${135/255} ${133/255} ${129/255} 1.0" />
   <!-- RAL 9010 - pure white  -->
   <xacro:property name="colour_kuka_ral_pure_white"       value="${241/255} ${236/255} ${255/255} 1.0" />
+  <!-- RAL 9016 - traffic white -->
+  <xacro:property name="colour_kuka_ral_traffic_white"    value="${241/255}  ${240/255} ${234/255} 1.0" />
 </robot>

File: kuka_resources/urdf/common_materials.xacro (robot description, xacro)
@@ -152,4 +152,9 @@
     </material>
   </xacro:macro>
+  <xacro:macro name="material_kuka_ral_gray_aluminium">
+    <material name="">
+      <color rgba="${colour_kuka_ral_gray_aluminium}"/>
+    </material>
+  </xacro:macro>
   <xacro:macro name="material_kuka_ral_pure_white">
     <material name="">
@@ -157,3 +162,8 @@
     </material>
   </xacro:macro>
+  <xacro:macro name="material_kuka_ral_traffic_white">
+    <material name="">
+      <color rgba="${colour_kuka_ral_traffic_white}"/>
+    </material>
+  </xacro:macro>
 </robot>
