Commit message: KR16-2: update visual colors, match appearance of KR16, use STL meshes instead of dae to allow coloring

File: kuka_kr16_support/urdf/kr16_2_macro.xacro (robot description, xacro)
@@ -1,4 +1,6 @@
 <?xml version="1.0"?>
 <robot xmlns:xacro="http://wiki.ros.org/xacro">
+  <xacro:include filename="$(find kuka_resources)/urdf/common_constants.xacro"/>
+  <xacro:include filename="$(find kuka_resources)/urdf/common_materials.xacro"/>
   <xacro:macro name="kuka_kr16_2" params="prefix">
     <!-- LINKS -->
@@ -13,6 +15,7 @@
         <origin xyz="0 0 0" rpy="0 0 0"/>
         <geometry>
-          <mesh filename="package://kuka_kr16_support/meshes/kr16_2/visual/base_link.dae" />
-        </geometry>
+          <mesh filename="package://kuka_kr16_support/meshes/kr16_2/visual/base_link.stl" />
+        </geometry>
+        <xacro:material_kuka_pedestal />
       </visual>
       <collision>
@@ -33,6 +36,7 @@
         <origin xyz="0 0 0" rpy="0 0 0"/>
         <geometry>
-          <mesh filename="package://kuka_kr16_support/meshes/kr16_2/visual/link_1.dae" />
-        </geometry>
+          <mesh filename="package://kuka_kr16_support/meshes/kr16_2/visual/link_1.stl" />
+        </geometry>
+        <xacro:material_kuka_orange />
       </visual>
       <collision>
@@ -53,6 +57,7 @@
         <origin xyz="0 0 0" rpy="0 0 0"/>
         <geometry>
-          <mesh filename="package://kuka_kr16_support/meshes/kr16_2/visual/link_2.dae"/>
-        </geometry>
+          <mesh filename="package://kuka_kr16_support/meshes/kr16_2/visual/link_2.stl"/>
+        </geometry>
+        <xacro:material_kuka_orange />
       </visual>
       <collision>
@@ -73,6 +78,7 @@
         <origin xyz="0 0 0" rpy="0 0 0"/>
         <geometry>
-          <mesh filename="package://kuka_kr16_support/meshes/kr16_2/visual/link_3.dae" />
-        </geometry>
+          <mesh filename="package://kuka_kr16_support/meshes/kr16_2/visual/link_3.stl" />
+        </geometry>
+        <xacro:material_kuka_orange />
       </visual>
       <collision>
@@ -93,6 +99,7 @@
         <origin xyz="0 0 0" rpy="0 0 0"/>
         <geometry>
-          <mesh filename="package://kuka_kr16_support/meshes/kr16_2/visual/link_4.dae" />
-        </geometry>
+          <mesh filename="package://kuka_kr16_support/meshes/kr16_2/visual/link_4.stl" />
+        </geometry>
+        <xacro:material_kuka_orange />
       </visual>
       <collision>
@@ -113,6 +120,7 @@
         <origin xyz="0 0 0" rpy="0 0 0"/>
         <geometry>
-          <mesh filename="package://kuka_kr16_support/meshes/kr16_2/visual/link_5.dae" />
-        </geometry>
+          <mesh filename="package://kuka_kr16_support/meshes/kr16_2/visual/link_5.stl" />
+        </geometry>
+        <xacro:material_kuka_orange />
       </visual>
       <collision>
@@ -133,6 +141,7 @@
         <origin xyz="0 0 0" rpy="0 0 0"/>
         <geometry>
-          <mesh filename="package://kuka_kr16_support/meshes/kr16_2/visual/link_6.dae" />
-        </geometry>
+          <mesh filename="package://kuka_kr16_support/meshes/kr16_2/visual/link_6.stl" />
+        </geometry>
+        <xacro:material_kuka_pedestal />
       </visual>
       <collision>

Commit message: WIP meshes don't match urdf origins

File: kuka_kr16_support/urdf/kr16_2_macro.xacro (robot description, xacro)
@@ -15,5 +15,5 @@
         <origin xyz="0 0 0" rpy="0 0 0"/>
         <geometry>
-          <mesh filename="package://kuka_kr16_support/meshes/kr16_2/visual/base_link.stl" />
+          <mesh filename="package://kuka_kr16_support/meshes/kr16/visual/base_link.stl" />
         </geometry>
         <xacro:material_kuka_pedestal />
@@ -22,5 +22,5 @@
         <origin xyz="0 0 0" rpy="0 0 0"/>
         <geometry>
-          <mesh filename="package://kuka_kr16_support/meshes/kr16_2/collision/base_link.stl" />
+          <mesh filename="package://kuka_kr16_support/meshes/kr16/collision/base_link.stl" />
         </geometry>
       </collision>
@@ -36,12 +36,12 @@
         <origin xyz="0 0 0" rpy="0 0 0"/>
         <geometry>
-          <mesh filename="package://kuka_kr16_support/meshes/kr16_2/visual/link_1.stl" />
-        </geometry>
-        <xacro:material_kuka_orange />
-      </visual>
-      <collision>
-        <origin xyz="0 0 0" rpy="0 0 0"/>
-        <geometry>
-          <mesh filename="package://kuka_kr16_support/meshes/kr16_2/collision/link_1.stl" />
+          <mesh filename="package://kuka_kr16_support/meshes/kr16/visual/link_1.stl" />
+        </geometry>
+        <xacro:material_kuka_orange />
+      </visual>
+      <collision>
+        <origin xyz="0 0 0" rpy="0 0 0"/>
+        <geometry>
+          <mesh filename="package://kuka_kr16_support/meshes/kr16/collision/link_1.stl" />
         </geometry>
       </collision>
@@ -57,12 +57,12 @@
         <origin xyz="0 0 0" rpy="0 0 0"/>
         <geometry>
-          <mesh filename="package://kuka_kr16_support/meshes/kr16_2/visual/link_2.stl"/>
-        </geometry>
-        <xacro:material_kuka_orange />
-      </visual>
-      <collision>
-        <origin xyz="0 0 0" rpy="0 0 0"/>
-        <geometry>
-          <mesh filename="package://kuka_kr16_support/meshes/kr16_2/collision/link_2.stl" />
+          <mesh filename="package://kuka_kr16_support/meshes/kr16/visual/link_2.stl"/>
+        </geometry>
+        <xacro:material_kuka_orange />
+      </visual>
+      <collision>
+        <origin xyz="0 0 0" rpy="0 0 0"/>
+        <geometry>
+          <mesh filename="package://kuka_kr16_support/meshes/kr16/collision/link_2.stl" />
         </geometry>
       </collision>
@@ -78,12 +78,12 @@
         <origin xyz="0 0 0" rpy="0 0 0"/>
         <geometry>
-          <mesh filename="package://kuka_kr16_support/meshes/kr16_2/visual/link_3.stl" />
-        </geometry>
-        <xacro:material_kuka_orange />
-      </visual>
-      <collision>
-        <origin xyz="0 0 0" rpy="0 0 0"/>
-        <geometry>
-          <mesh filename="package://kuka_kr16_support/meshes/kr16_2/collision/link_3.stl" />
+          <mesh filename="package://kuka_kr16_support/meshes/kr16/visual/link_3.stl" />
+        </geometry>
+        <xacro:material_kuka_orange />
+      </visual>
+      <collision>
+        <origin xyz="0 0 0" rpy="0 0 0"/>
+        <geometry>
+          <mesh filename="package://kuka_kr16_support/meshes/kr16/collision/link_3.stl" />
         </geometry>
       </collision>
@@ -99,12 +99,12 @@
         <origin xyz="0 0 0" rpy="0 0 0"/>
         <geometry>
-          <mesh filename="package://kuka_kr16_support/meshes/kr16_2/visual/link_4.stl" />
-        </geometry>
-        <xacro:material_kuka_orange />
-      </visual>
-      <collision>
-        <origin xyz="0 0 0" rpy="0 0 0"/>
-        <geometry>
-          <mesh filename="package://kuka_kr16_support/meshes/kr16_2/collision/link_4.stl" />
+          <mesh filename="package://kuka_kr16_support/meshes/kr16/visual/link_4.stl" />
+        </geometry>
+        <xacro:material_kuka_orange />
+      </visual>
+      <collision>
+        <origin xyz="0 0 0" rpy="0 0 0"/>
+        <geometry>
+          <mesh filename="package://kuka_kr16_support/meshes/kr16/collision/link_4.stl" />
         </geometry>
       </collision>
@@ -120,12 +120,12 @@
         <origin xyz="0 0 0" rpy="0 0 0"/>
         <geometry>
-          <mesh filename="package://kuka_kr16_support/meshes/kr16_2/visual/link_5.stl" />
-        </geometry>
-        <xacro:material_kuka_orange />
-      </visual>
-      <collision>
-        <origin xyz="0 0 0" rpy="0 0 0"/>
-        <geometry>
-          <mesh filename="package://kuka_kr16_support/meshes/kr16_2/collision/link_5.stl" />
+          <mesh filename="package://kuka_kr16_support/meshes/kr16/visual/link_5.stl" />
+        </geometry>
+        <xacro:material_kuka_orange />
+      </visual>
+      <collision>
+        <origin xyz="0 0 0" rpy="0 0 0"/>
+        <geometry>
+          <mesh filename="package://kuka_kr16_support/meshes/kr16/collision/link_5.stl" />
         </geometry>
       </collision>
@@ -141,5 +141,5 @@
         <origin xyz="0 0 0" rpy="0 0 0"/>
         <geometry>
-          <mesh filename="package://kuka_kr16_support/meshes/kr16_2/visual/link_6.stl" />
+          <mesh filename="package://kuka_kr16_support/meshes/kr16/visual/link_6.stl" />
         </geometry>
         <xacro:material_kuka_pedestal />
@@ -148,5 +148,5 @@
         <origin xyz="0 0 0" rpy="0 0 0"/>
         <geometry>
-          <mesh filename="package://kuka_kr16_support/meshes/kr16_2/collision/link_6.stl" />
+          <mesh filename="package://kuka_kr16_support/meshes/kr16/collision/link_6.stl" />
         </geometry>
       </collision>
