Commit message: Add KR210 R2700-prime, rm kr210l150.urdf
fix whitespace

File: kuka_kr210_support/urdf/kr210_r2700-prime_macro.xacro (robot description, xacro)
@@ -1,155 +1,139 @@
 <?xml version="1.0"?>
 <robot xmlns:xacro="http://wiki.ros.org/xacro">
-  <xacro:include filename="$(find kuka_resources)/urdf/common_constants.xacro"/>
-  <xacro:include filename="$(find kuka_resources)/urdf/common_materials.xacro"/>
-  <xacro:macro name="kuka_kr210_r3100-2" params="prefix">
-    <!-- LINKS -->
-    <!-- base link -->
+  <xacro:macro name="kuka_kr210_r2700-prime" params="prefix">
+    <xacro:include filename="$(find kuka_resources)/urdf/common_materials.xacro"/>
     <link name="${prefix}base_link">
       <visual>
-        <origin rpy="0 0 0" xyz="0 0 0"/>
+        <origin xyz="0 0 0" rpy="0 0 0" />
         <geometry>
-          <mesh filename="package://kuka_kr210_support/meshes/kr210_r3100-2/visual/base_link.stl" />
+          <mesh filename="package://kuka_kr210_support/meshes/kr210_r2700-prime/visual/base_link.stl"  />
         </geometry>
         <xacro:material_kuka_pedestal />
       </visual>
       <collision>
-        <origin rpy="0 0 0" xyz="0 0 0"/>
+        <origin xyz="0 0 0" rpy="0 0 0" />
         <geometry>
-          <mesh filename="package://kuka_kr210_support/meshes/kr210_r3100-2/collision/base_link.stl" />
+          <mesh filename="package://kuka_kr210_support/meshes/kr210_r2700-prime/collision/base_link.stl"  />
         </geometry>
       </collision>
     </link>
-    <!-- link 1 (A1) -->
     <link name="${prefix}link_1">
       <visual>
-        <origin xyz="0 0 0" rpy="0 0 0"/>
+        <origin xyz="0 0 0" rpy="0 0 0" />
         <geometry>
-          <mesh filename="package://kuka_kr210_support/meshes/kr210_r3100-2/visual/link_1.stl" />
+          <mesh filename="package://kuka_kr210_support/meshes/kr210_r2700-prime/visual/link_1.stl"  />
         </geometry>
         <xacro:material_kuka_orange />
       </visual>
       <collision>
-        <origin xyz="0 0 0" rpy="0 0 0"/>
+        <origin xyz="0 0 0" rpy="0 0 0" />
         <geometry>
-          <mesh filename="package://kuka_kr210_support/meshes/kr210_r3100-2/collision/link_1.stl" />
+          <mesh filename="package://kuka_kr210_support/meshes/kr210_r2700-prime/collision/link_1.stl"  />
         </geometry>
       </collision>
     </link>
-    <!-- link 2 -->
     <link name="${prefix}link_2">
       <visual>
-        <origin xyz="0 0 0" rpy="0 0 0"/>
+        <origin xyz="0 0 0" rpy="0 0 0" />
         <geometry>
-          <mesh filename="package://kuka_kr210_support/meshes/kr210_r3100-2/visual/link_2.stl"/>
+          <mesh filename="package://kuka_kr210_support/meshes/kr210_r2700-prime/visual/link_2.stl"  />
         </geometry>
         <xacro:material_kuka_orange />
       </visual>
       <collision>
-        <origin xyz="0 0 0" rpy="0 0 0"/>
+        <origin xyz="0 0 0" rpy="0 0 0" />
         <geometry>
-          <mesh filename="package://kuka_kr210_support/meshes/kr210_r3100-2/collision/link_2.stl"  />
+          <mesh filename="package://kuka_kr210_support/meshes/kr210_r2700-prime/collision/link_2.stl"  />
         </geometry>
       </collision>
     </link>
-    <!-- link 3 -->
     <link name="${prefix}link_3">
       <visual>
-        <origin xyz="0 0 0" rpy="0 0 0"/>
+        <origin xyz="0 0 0" rpy="0 0 0" />
         <geometry>
-          <mesh filename="package://kuka_kr210_support/meshes/kr210_r3100-2/visual/link_3.stl" />
+          <mesh filename="package://kuka_kr210_support/meshes/kr210_r2700-prime/visual/link_3.stl"  />
         </geometry>
         <xacro:material_kuka_orange />
       </visual>
       <collision>
-        <origin xyz="0 0 0" rpy="0 0 0"/>
+        <origin xyz="0 0 0" rpy="0 0 0" />
         <geometry>
-          <mesh filename="package://kuka_kr210_support/meshes/kr210_r3100-2/collision/link_3.stl"  />
+          <mesh filename="package://kuka_kr210_support/meshes/kr210_r2700-prime/collision/link_3.stl"  />
         </geometry>
       </collision>
     </link>
-    <!-- link 4 -->
     <link name="${prefix}link_4">
       <visual>
-        <origin xyz="0 0 0" rpy="0 0 0"/>
+        <origin xyz="0 0 0" rpy="0 0 0" />
         <geometry>
-          <mesh filename="package://kuka_kr210_support/meshes/kr210_r3100-2/visual/link_4.stl" />
+          <mesh filename="package://kuka_kr210_support/meshes/kr210_r2700-prime/visual/link_4.stl"  />
         </geometry>
         <xacro:material_kuka_orange />
       </visual>
       <collision>
-        <origin xyz="0 0 0" rpy="0 0 0"/>
+        <origin xyz="0 0 0" rpy="0 0 0" />
         <geometry>
-          <mesh filename="package://kuka_kr210_support/meshes/kr210_r3100-2/collision/link_4.stl"  />
+          <mesh filename="package://kuka_kr210_support/meshes/kr210_r2700-prime/collision/link_4.stl"  />
         </geometry>
       </collision>
     </link>
-    <!-- link 5 -->
     <link name="${prefix}link_5">
       <visual>
-        <origin xyz="0 0 0" rpy="0 0 0"/>
+        <origin xyz="0 0 0" rpy="0 0 0" />
         <geometry>
-          <mesh filename="package://kuka_kr210_support/meshes/kr210_r3100-2/visual/link_5.stl" />
+          <mesh filename="package://kuka_kr210_support/meshes/kr210_r2700-prime/visual/link_5.stl"  />
         </geometry>
         <xacro:material_kuka_orange />
       </visual>
       <collision>
-        <origin xyz="0 0 0" rpy="0 0 0"/>
+        <origin xyz="0 0 0" rpy="0 0 0" />
         <geometry>
-          <mesh filename="package://kuka_kr210_support/meshes/kr210_r3100-2/collision/link_5.stl" />
+          <mesh filename="package://kuka_kr210_support/meshes/kr210_r2700-prime/collision/link_5.stl"  />
         </geometry>
       </collision>
     </link>
-    <!-- link 6 -->
     <link name="${prefix}link_6">
       <visual>
-        <origin xyz="0 0 0" rpy="0 0 0"/>
+        <origin xyz="0 0 0" rpy="0 0 0" />
         <geometry>
-          <mesh filename="package://kuka_kr210_support/meshes/kr210_r3100-2/visual/link_6.stl" />
+          <mesh filename="package://kuka_kr210_support/meshes/kr210_r2700-prime/visual/link_6.stl"  />
         </geometry>
-        <xacro:material_kuka_orange />
+        <xacro:material_kuka_pedestal />
       </visual>
       <collision>
-        <origin xyz="0 0 0" rpy="0 0 0"/>
+        <origin xyz="0 0 0" rpy="0 0 0" />
         <geometry>
-          <mesh filename="package://kuka_kr210_support/meshes/kr210_r3100-2/collision/link_6.stl" />
+          <mesh filename="package://kuka_kr210_support/meshes/kr210_r2700-prime/collision/link_6.stl"  />
         </geometry>
       </collision>
     </link>
-    <!-- END LINKS -->
-    <!-- JOINTS -->
-    <!-- joint 1 (A1) -->
     <joint name="${prefix}joint_a1" type="revolute">
-      <origin xyz="0 0 0.645" rpy="0 0 0"/>
+      <origin xyz="0 0 0.675" rpy="0 0 0"/>
       <parent link="${prefix}base_link"/>
       <child link="${prefix}link_1"/>
       <axis xyz="0 0 -1"/>
-      <limit effort="0" lower="${radians(-185)}" upper="${radians(185)}" velocity="${radians(105)}"/>
+      <limit lower="${radians(-185)}" upper="${radians(185)}" effort="0" velocity="${radians(105)}"/>
     </joint>
-    <!-- joint 2 (A2) -->
     <joint name="${prefix}joint_a2" type="revolute">
-      <origin xyz="0.33 0 0" rpy="0 0 0"/>
+      <origin xyz="0.350 0 0" rpy="0 0 0"/>
       <parent link="${prefix}link_1"/>
       <child link="${prefix}link_2"/>
       <axis xyz="0 1 0"/>
-      <limit effort="0" lower="${radians(-140)}" upper="${radians(-5)}" velocity="${radians(94)}"/>
+      <limit lower="${radians(-140)}" upper="${radians(-5)}" effort="0" velocity="${radians(107)}"/>
     </joint>
-    <!-- joint 3 (A3) -->
     <joint name="${prefix}joint_a3" type="revolute">
-      <origin xyz="1.350 0 0" rpy="0 0 0"/>
+      <origin xyz="1.150 0 0.0" rpy="0 0 0"/>
       <parent link="${prefix}link_2"/>
       <child link="${prefix}link_3"/>
       <axis xyz="0 1 0"/>
-      <limit effort="0" lower="${radians(-120)}" upper="${radians(168)}" velocity="${radians(100)}"/>
+      <limit lower="${radians(-120)}" upper="${radians(155)}" effort="0" velocity="${radians(114)}"/>
     </joint>
-    <!-- joint 4 (A4) -->
     <joint name="${prefix}joint_a4" type="revolute">
-      <origin xyz="1.420 0 0.115" rpy="0 0 0"/>
+      <origin xyz="1.200 0 -0.041" rpy="0 0 0"/>
       <parent link="${prefix}link_3"/>
       <child link="${prefix}link_4"/>
       <axis xyz="-1 0 0"/>
-      <limit effort="0" lower="${radians(-350)}" upper="${radians(350)}" velocity="${radians(136)}"/>
+      <limit lower="${radians(-350)}" upper="${radians(350)}" effort="0" velocity="${radians(136)}"/>
     </joint>
-    <!-- joint 5 (A5) -->
     <joint name="${prefix}joint_a5" type="revolute">
       <origin xyz="0 0 0" rpy="0 0 0"/>
@@ -157,7 +141,6 @@
       <child link="${prefix}link_5"/>
       <axis xyz="0 1 0"/>
-      <limit effort="0" lower="${radians(-122.5)}" upper="${radians(122.5)}" velocity="${radians(129)}"/>
+      <limit lower="${radians(-122.5)}" upper="${radians(122.5)}" effort="0" velocity="${radians(129)}"/>
     </joint>
-    <!-- joint 6 (A6) -->
     <joint name="${prefix}joint_a6" type="revolute">
       <origin xyz="0.240 0 0" rpy="0 0 0"/>
@@ -165,7 +148,6 @@
       <child link="${prefix}link_6"/>
       <axis xyz="-1 0 0"/>
-      <limit effort="0" lower="${radians(-350)}" upper="${radians(350)}" velocity="${radians(206)}"/>
+      <limit lower="${radians(-350)}" upper="${radians(350)}" effort="0" velocity="${radians(206)}"/>
     </joint>
-    <!-- END JOINTS -->
     <!-- ROS-Industrial 'base' frame: base_link to KUKA $ROBROOT coordinate system transform -->
     <link name="${prefix}base" />
@@ -185,6 +167,6 @@
     <!-- This frame corresponds to the $FLANGE coordinate system in KUKA KRC controllers. -->
     <link name="${prefix}tool0"/>
-    <joint name="${prefix}joint_a6-tool0" type="fixed">
-      <parent link="${prefix}link_6"/>
+    <joint name="${prefix}flange-tool0" type="fixed">
+      <parent link="${prefix}flange"/>
       <child link="${prefix}tool0"/>
       <origin xyz="0 0 0" rpy="0 ${radians(90)} 0"/>
